File: VBC-HW/Victor-Brushless-Controller.kicad_pcb (KiCad board)
At the start: 2 copper layers, 0 parts

Commit message: Ready to tetris
Parts:
- added ?: , , F.Cu at (198.5, 111.5)
- added ?: , , F.Cu at (160.5, 76.5)
- added ?: , , F.Cu at (198.5, 76.5)
- added C1: 1nF, 0402B102K500NT:0402B102K500NT, F.Cu at (96.5, 104.7)
- added C10: 1uF, CL05A105KA5NQNC:CL05A105KA5NQNC, F.Cu at (100.0, 104.7)
- added C11: 1uF, CL05A105KA5NQNC:CL05A105KA5NQNC, F.Cu at (100.0, 106.9)
- added C12: 100nF, CL05B104KO5NNNC:CL05B104KO5NNNC, F.Cu at (100.0, 109.0)
- added C13: 1nF, 0402B102K500NT:0402B102K500NT, F.Cu at (100.0, 111.2)
- added C14: 10uF, CL05A106MQ5NUNC:CL05A106MQ5NUNC, F.Cu at (100.0, 113.3)
- added C15: 10uF, CL05B104KO5NNNC:CL05B104KO5NNNC, F.Cu at (103.5, 104.7)
- added C16: 100nF, CL05B104KO5NNNC:CL05B104KO5NNNC, F.Cu at (103.5, 106.9)
- added C17: 22uF, CL10A226MQ8NRNC:CL10A226MQ8NRNC, F.Cu at (117.0, 96.7)
- added C18: 10uF, CL10A106MA8NRNC:CL10A106MA8NRNC, F.Cu at (117.0, 99.3)
- added C19: 1uF, CL10A105KB8NNNC:CL10A105KB8NNNC, F.Cu at (117.0, 102.0)
- added C2: 1nF, 0402B102K500NT:0402B102K500NT, F.Cu at (96.5, 106.9)
- added C20: 10uF, GRM21BR61H106KE43L:GRM21BR61H106KE43L, F.Cu at (72.5, 97.1)
- added C21: 100nF, CL05B104KO5NNNC:CL05B104KO5NNNC, F.Cu at (103.5, 109.0)
- added C22: 10uF, GRM21BR61H106KE43L:GRM21BR61H106KE43L, F.Cu at (72.5, 100.0)
- added C23: 10uF, GRM21BR61H106KE43L:GRM21BR61H106KE43L, F.Cu at (72.5, 103.0)
- added C24: 10uF, GRM21BR61H106KE43L:GRM21BR61H106KE43L, F.Cu at (72.5, 105.9)
- added C25: 10uF, GRM21BR61H106KE43L:GRM21BR61H106KE43L, F.Cu at (77.5, 94.1)
- added C26: 10uF, GRM21BR61H106KE43L:GRM21BR61H106KE43L, F.Cu at (77.5, 97.1)
- added C27: 10uF, GRM21BR61H106KE43L:GRM21BR61H106KE43L, F.Cu at (77.5, 100.0)
- added C3: 1nF, 0402B102K500NT:0402B102K500NT, F.Cu at (96.5, 109.0)
- added C30: 100nF, CL05B104KO5NNNC:CL05B104KO5NNNC, F.Cu at (103.5, 111.2)
- added C31: 10uF, GRM21BR61H106KE43L:GRM21BR61H106KE43L, F.Cu at (77.5, 103.0)
- added C32: 10uF, GRM21BR61H106KE43L:GRM21BR61H106KE43L, F.Cu at (77.5, 105.9)
- added C33: 10uF, GRM21BR61H106KE43L:GRM21BR61H106KE43L, F.Cu at (82.6, 94.1)
- added C34: 10uF, GRM21BR61H106KE43L:GRM21BR61H106KE43L, F.Cu at (82.6, 97.1)
- added C35: 10uF, GRM21BR61H106KE43L:GRM21BR61H106KE43L, F.Cu at (82.6, 100.0)
- added C36: 10uF, GRM21BR61H106KE43L:GRM21BR61H106KE43L, F.Cu at (82.6, 103.0)
- added C37: 10uF, 1206X106M500NT:1206X106M500NT, F.Cu at (103.0, 72.3)
- added C38: 10uF, 1206X106M500NT:1206X106M500NT, F.Cu at (103.0, 75.7)
- added C39: 10uF, GRM21BR61H106KE43L:GRM21BR61H106KE43L, F.Cu at (82.6, 105.9)
- added C4: 1uF, CL05A105KA5NQNC:CL05A105KA5NQNC, F.Cu at (96.5, 111.2)
- added C5: 4.7uF, 1206B475K500NT:1206B475K500NT, F.Cu at (103.0, 65.7)
- added C6: 1uF, CL05A105KA5NQNC:CL05A105KA5NQNC, F.Cu at (96.5, 113.3)
- added C7: 2.2uF, CL31B225KBHNNNE:CL31B225KBHNNNE, F.Cu at (103.0, 69.0)
- added C8: 47nF, CL21B473KCFNNNE:CL21B473KCFNNNE, F.Cu at (72.5, 94.1)
- added C9: 47nF, CL10B473KB8NNNC:CL10B473KB8NNNC, F.Cu at (117.0, 94.0)
- added D1: B230A-13-F, B230A-13-F:B230A-13-F, F.Cu at (73.5, 109.4)
- added D2: SMA6J24A-TR, SMA6J24A:SMA6J24A, F.Cu at (88.8, 109.8)
- added H1: Extra GPIOs, Connector_PinHeader_2.54mm:PinHeader_1x02_P2.54mm_Vertical, F.Cu at (114.0, 86.5)
- added H2: Programming UART, Connector_PinHeader_2.54mm:PinHeader_1x04_P2.54mm_Vertical, F.Cu at (108.1, 95.0)
- added H3: Extra Sources, Connector_PinHeader_2.54mm:PinHeader_1x04_P2.54mm_Vertical, F.Cu at (112.7, 95.0)
- added J1: i2c QWIIC, Connector_JST:JST_GH_BM04B-GHS-TBT_1x04-1MP_P1.25mm_Vertical, F.Cu at (111.4, 67.8)
- added JP1: SolderJumper, Jumper:SolderJumper-2_P1.3mm_Open_Pad1.0x1.5mm, F.Cu at (72.1, 113.1)
- added L1: 15uH, PIS3D18P-150M-T:PIS3D18P-150M-T, F.Cu at (94.7, 79.8)
- added LED1: Red, KT-0603R:KT-0603R, F.Cu at (109.7, 85.5)
- added LED2: Blue, 19-217:19-217, F.Cu at (109.7, 88.2)
- added LED3: Yellow, 19-213:19-213, F.Cu at (109.7, 90.8)
- added P1: PVDD, Power_Connector:Power_Connector, F.Cu at (108.2, 107.4)
- added P2: GND, Power_Connector:Power_Connector, F.Cu at (108.2, 112.4)
- added PA1: Phase, BLDC_Connector:BLDC_Connector, F.Cu at (97.6, 58.6)
- added PB1: Phase, BLDC_Connector:BLDC_Connector, F.Cu at (97.6, 62.6)
- added PC1: Phase, BLDC_Connector:BLDC_Connector, F.Cu at (97.6, 66.6)
- added Q1: TPH4R008NH, TPH4R008NH,L1Q(M:TPH4R008NH,L1Q(M, F.Cu at (73.1, 88.1)
- added Q2: TPH4R008NH, TPH4R008NH,L1Q(M:TPH4R008NH,L1Q(M, F.Cu at (79.4, 88.1)
- added Q3: TPH4R008NH, TPH4R008NH,L1Q(M:TPH4R008NH,L1Q(M, F.Cu at (85.7, 88.1)
- added Q4: TPH4R008NH, TPH4R008NH,L1Q(M:TPH4R008NH,L1Q(M, F.Cu at (92.0, 88.1)
- added Q5: TPH4R008NH, TPH4R008NH,L1Q(M:TPH4R008NH,L1Q(M, F.Cu at (98.2, 88.1)
- added Q6: TPH4R008NH, TPH4R008NH,L1Q(M:TPH4R008NH,L1Q(M, F.Cu at (104.5, 88.1)
- added R1: 0.002, CUM2512-24FR002:CUM2512-24FR002, F.Cu at (89.9, 95.2)
- added R10: 3k3, 0402WGF3301TCE:0402WGF3301TCE, F.Cu at (110.7, 77.0)
- added R11: 10k, 0402WGF1002TCE:0402WGF1002TCE, F.Cu at (110.7, 79.2)
- added R12: 110k, RC0402FR-07110KL:RC0402FR-07110KL, F.Cu at (113.7, 72.7)
- added R13: 33k, 0402WGF3302TCE:0402WGF3302TCE, F.Cu at (113.7, 74.9)
- added R15: 2k2, 0402WGF2201TCE:0402WGF2201TCE, F.Cu at (113.7, 77.0)
- added R2: 0.002, CUM2512-24FR002:CUM2512-24FR002, F.Cu at (89.9, 100.3)
- added R3: 0.002, CUM2512-24FR002:CUM2512-24FR002, F.Cu at (89.9, 105.4)
- added R4: 330, 0402WGF3300TCE:0402WGF3300TCE, F.Cu at (107.7, 72.7)
- added R5: 10k, 0402WGF1002TCE:0402WGF1002TCE, F.Cu at (107.7, 74.9)
- added R6: 10k, 0402WGF1002TCE:0402WGF1002TCE, F.Cu at (107.7, 77.0)
- added R7: 100, 0402WGF1000TCE:0402WGF1000TCE, F.Cu at (107.7, 79.2)
- added R8: 330, 0402WGF3300TCE:0402WGF3300TCE, F.Cu at (110.7, 72.7)
- added R9: 33k, 0402WGF3302TCE:0402WGF3302TCE, F.Cu at (110.7, 74.9)
- added REF**: MountingHole_2.7mm_M2.5_DIN965_Pad, MountingHole:MountingHole_2.7mm_M2.5_DIN965_Pad, F.Cu at (160.5, 111.5)
- added SW1: SW_SPST, TS342A2P-WZ:TS342A2P-WZ, F.Cu at (94.5, 70.5)
- added SW2: SW_SPST, TS342A2P-WZ:TS342A2P-WZ, F.Cu at (94.5, 74.8)
- added U1: DRV8305NQPHPRQ1, DRV8305NQPHPRQ1:DRV8305NQPHPRQ1, F.Cu at (100.2, 98.2)
- added U2: ESP-WROOM-32E, ESP-WROOM-32E:ESP-WROOM-32E, F.Cu at (80.6, 73.6)
- added U3: LMR14010ADDCR, LMR14010ADDCR:LMR14010ADDCR, F.Cu at (79.5, 109.6)
- added U5: STLM20W87F, STLM20W87F:STLM20W87F, F.Cu at (101.9, 79.4)
- added U6: External SPI, Connector_JST:JST_GH_BM06B-GHS-TBT_1x06-1MP_P1.25mm_Vertical, F.Cu at (106.4, 60.2)
- added U7: AS5047P-ATSM_C962063, AS5047P-ATSM:AS5047P-ATSM, F.Cu at (113.9, 109.1)
