File: VBC-HW/Victor-Brushless-Controller.kicad_pcb (KiCad board)
At the start: 4 copper layers, 44 x 44 mm, 85 parts, among them J1 i2c/UART, P1 V+, P2 GND, Q1 TPH4R008NH, Q2 TPH4R008NH, Q3 TPH4R008NH, Q4 TPH4R008NH, Q5 TPH4R008NH, Q6 TPH4R008NH, SW1 BOOT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

Commit message: Finished all connections
Parts:
- moved C37 0.35 mm to (191.6, 98.0)
- moved C4 0.34 mm to (158.3, 97.3)
Connections:
- J1 pad 1: GND -> IO22
- J1 pad 2: 3V3A -> IO21
- J1 pad 3: IO21 -> 3V3A
- J1 pad 4: IO22 -> GND
- U1 pad 1: EN I02 -> EN IO2
- U6 pad 1: 3V3A -> SDO MISO19
- U6 pad 2: GND -> SDI MOSI23
- U6 pad 3: EXTCS IO12 -> SCLK IO18
- U6 pad 4: SCLK IO18 -> EXTCS IO12
- U6 pad 5: SDI MOSI23 -> GND
- U6 pad 6: SDO MISO19 -> 3V3A
Routing:
- net GND: track 104.4 -> 189.4 mm
- net SCLK IO18: track 1.57 -> 74.1 mm, vias 1 -> 2
- net SDO MISO19: track 1.56 -> 65.8 mm, vias 1 -> 4
- net BOOT IO0: track 7.23 -> 67.1 mm, vias 2 -> 3
- net RESET EN: track 8.67 -> 58.1 mm
- net SDI MOSI23: track 25.8 -> 73.4 mm, vias 2 -> 3
- net EXTCS IO12: track 1.35 -> 45.6 mm, vias 1 -> 3
- net SO3 IO36: track 6.55 -> 48.7 mm, vias 1 -> 2
- net NSCS SS05: track 1.56 -> 41.8 mm, vias 1 -> 2
- net SO2 IO35: track 1.80 -> 41.1 mm, vias 1 -> 2
- net SO1 IO34: track 1.77 -> 39.4 mm, vias 1 -> 2
- net 3V3A: track 30.0 -> 65.9 mm, vias 9 -> 13
- net nFault IO4: track 14.9 -> 48.9 mm, vias 3 -> 4
- net INLx IO14: track 1.56 -> 31.8 mm, vias 1 -> 4
- net /SLA: track 25.4 -> 54.8 mm, vias 8 -> 10
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- added copper zone on In2.Cu, net 3V3A
- added copper zone on B.Cu, net VCC
- added copper zone on In2.Cu, net VCC
Other:
- board text added: "Victor Brushless Controller For the Cabrestrante S. Actuator"

Commit message: Fully finished board
Routing:
- net 3V3: track 25.8 -> 28.4 mm
- net 3V3A: track 65.9 -> 67.8 mm
Other:
- board text added: "3V3"
- board text added: "A"
- board text added: "B"
- board text added: "BOOT"
- board text added: "Based on DAGOR 2.7"
- board text added: "C"
- board text added: "En"
- board text added: "GND"
- board text added: "GPIOs"
- board text added: "IO0"
- board text added: "IO12"
- board text added: "IO21"
- board text added: "IO22"
- board text added: "Prog"
- board text added: "RESET"
- board text added: "RX0"
- board text added: "TX0"
- board text added: "V+"
- board text added: "VD"
- board text added: "⌀ M2.5 ⁘ 35x35mm □ 44x44mm"
